File: pcb/numpad_v1a.brd (EAGLE design)
At the start: 98 x 98 mm, 87 parts, among them IC1 ATMEGA32U4-MU, IC2 IS31FL3731-SALS2, SW1 EVQP2, X1 16MHz

Commit message: fix(schematic): Corrected LED driver part number
Parts:
- IC2: value IS31FL3731-SALS2 -> IS31FL3731-QFLS2
Changed lines of the file:
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@@
 <attribute name="VALUE" x="85.9" y="93.3" size="1.27" layer="28" rot="MR180"/>
 </element>
-<element name="IC2" library="microbuilder" package="QFN28_4MM_0.4MM" value="IS31FL3731-SALS2" x="87" y="67" smashed="yes" rot="MR0">
+<element name="IC2" library="microbuilder" package="QFN28_4MM_0.4MM" value="IS31FL3731-QFLS2" x="87" y="67" smashed="yes" rot="MR0">
 <attribute name="NAME" x="88.25" y="69.8" size="1.27" layer="26" font="vector" ratio="20" rot="MR0"/>
 <attribute name="VALUE" x="94.4" y="71.35" size="0.4064" layer="28" ratio="10" rot="MR0"/>
